File: board/board.kicad_sch (KiCad schematic)
At the start: 1 part

Commit message: initial
Parts:
- added J1, J2: Conn_01x02_Socket, TerminalBlock:TerminalBlock_MaiXu_MX126-5.0-02P_1x02_P5.00mm, symbol Connector:Conn_01x02_Socket
- added R1: 100k, Resistor_SMD:R_0603_1608Metric, symbol Device:R_Small
- added TPM1: Mode, TestPoint:TestPoint_Pad_2.0x2.0mm, symbol Connector:TestPoint
Connections:
- net GND: now also J1.1 (Pin_1), J2.1 (Pin_1)
- new net 8A_DCDC/5V: J1.2 (Pin_2)
- new net 8A_DCDC/En: R1.2
- new net 8A_DCDC/In: J2.2 (Pin_2), R1.1
- new net 8A_DCDC/Mode: TPM1.1
Other:
- sheet implementation renamed 8A_DCDC
- sheet 8A_DCDC: file implementation.kicad_sch -> 8A_DCDC.kicad_sch
- sheet 8A_DCDC ports: added 5V, En, In, Mode; removed none
- note removed: "Input connectors go here"
- note removed: "Output connectors go here"
